File: Motor_ECU.sch (KiCad schematic (older format))
At the start: 28 parts, among them J1 Conn_01x04, J2 Conn_01x04, J3 Conn_01x02, J4 Debug, J5 Conn_01x02, U1 IFX9201SG, U2 TLE4964, U3 XMC1404_F064, U4 TLE7251, U5 LM35-D

Commit message: Clean up in the symbol libs
Parts:
- C1, C10, C11, C12, C13, C14, C2, C3, C4, C5, C6, C7, C8, C9: symbol Wheel_ECU-rescue:C -> Motor_ECU-rescue:C-Wheel_ECU-rescue
- D1, D2: symbol Wheel_ECU-rescue:TVS_Diode -> Motor_ECU-rescue:TVS_Diode-Wheel_ECU-rescue
- J1, J2: symbol Wheel_ECU-rescue:Conn_01x04 -> Motor_ECU-rescue:Conn_01x04-Wheel_ECU-rescue
- J3: symbol Wheel_ECU-rescue:Conn_01x02 -> Motor_ECU-rescue:Conn_01x02-Wheel_ECU-rescue
- J4: symbol Wheel_ECU-rescue:Conn_02x04_Odd_Even -> Motor_ECU-rescue:Conn_02x04_Odd_Even-Wheel_ECU-rescue
- U1: symbol wheel_ecu:IFX9201SG -> motor_drivers:IFX9201SG
- U2: symbol Wheel_ECU-rescue:TLE4964 -> sensors:TLE4964
- U3: symbol Wheel_ECU-rescue:XMC1404_F064 -> mcu:XMC1404_F064
- U4: symbol Wheel_ECU-rescue:TLE7251 -> transceivers:TLE7251
Changed lines of the file:
@@
 $EndDescr
 $Comp
-L Wheel_ECU-rescue:XMC1404_F064 U3
+L mcu:XMC1404_F064 U3
 U 1 1 5BFABA33
 P 3700 3400
@@
 $EndComp
 $Comp
-L Wheel_ECU-rescue:TLE7251 U4
+L transceivers:TLE7251 U4
 U 1 1 5BFABC56
 P 9250 950
@@
 $EndComp
 $Comp
-L Wheel_ECU-rescue:TLE4964 U2
+L sensors:TLE4964 U2
 U 1 1 5BFAD6F2
 P 6750 2700
@@
 $EndComp
 $Comp
-L Wheel_ECU-rescue:Conn_02x04_Odd_Even J4
+L Motor_ECU-rescue:Conn_02x04_Odd_Even-Wheel_ECU-rescue J4
 U 1 1 5BFAD803
 P 6250 1700
@@
 $EndComp
 $Comp
-L Wheel_ECU-rescue:Conn_01x02 J3
+L Motor_ECU-rescue:Conn_01x02-Wheel_ECU-rescue J3
 U 1 1 5BFAD8F5
 P 4700 2500
@@
 $EndComp
 $Comp
-L Wheel_ECU-rescue:C C2
+L Motor_ECU-rescue:C-Wheel_ECU-rescue C2
 U 1 1 5BFADA57
 P 5850 3150
@@
 $EndComp
 $Comp
-L Wheel_ECU-rescue:C C4
+L Motor_ECU-rescue:C-Wheel_ECU-rescue C4
 U 1 1 5BFADB7C
 P 8450 1800
@@
 $EndComp
 $Comp
-L Wheel_ECU-rescue:C C1
+L Motor_ECU-rescue:C-Wheel_ECU-rescue C1
 U 1 1 5BFADC1D
 P 8250 5700
@@
 $EndComp
 $Comp
-L Wheel_ECU-rescue:C C3
+L Motor_ECU-rescue:C-Wheel_ECU-rescue C3
 U 1 1 5BFADD3C
 P 2150 4050
@@
 $EndComp
 $Comp
-L Wheel_ECU-rescue:C C5
+L Motor_ECU-rescue:C-Wheel_ECU-rescue C5
 U 1 1 5BFAE74E
 P 10250 2050
@@
 $EndComp
 $Comp
-L Wheel_ECU-rescue:TVS_Diode D1
+L Motor_ECU-rescue:TVS_Diode-Wheel_ECU-rescue D1
 U 1 1 5BFB197A
 P 7850 6000
@@
 $EndComp
 $Comp
-L Wheel_ECU-rescue:GND #PWR02
+L Motor_ECU-rescue:GND-Wheel_ECU-rescue #PWR02
 U 1 1 5BFB2839
 P 2400 2050
@@
 $EndComp
 $Comp
-L Wheel_ECU-rescue:GND #PWR03
+L Motor_ECU-rescue:GND-Wheel_ECU-rescue #PWR03
 U 1 1 5BFC2172
 P 8250 6050
@@
 $EndComp
 $Comp
-L Wheel_ECU-rescue:+5V #PWR04
+L Motor_ECU-rescue:+5V-Wheel_ECU-rescue #PWR04
 U 1 1 5BFC2551
 P 2300 3600
@@
 $EndComp
 $Comp
-L Wheel_ECU-rescue:GND #PWR05
+L Motor_ECU-rescue:GND-Wheel_ECU-rescue #PWR05
 U 1 1 5BFC25D3
 P 950 4450
@@
 CAN+
 $Comp
-L Wheel_ECU-rescue:GND #PWR06
+L Motor_ECU-rescue:GND-Wheel_ECU-rescue #PWR06
 U 1 1 5BFC2CC6
 P 9750 6000
@@
 $EndComp
 $Comp
-L Wheel_ECU-rescue:+5V #PWR07
+L Motor_ECU-rescue:+5V-Wheel_ECU-rescue #PWR07
 U 1 1 5BFC2D01
 P 9150 5400
@@
 $EndComp
 $Comp
-L Wheel_ECU-rescue:GND #PWR08
+L Motor_ECU-rescue:GND-Wheel_ECU-rescue #PWR08
 U 1 1 5BFC30F3
 P 6000 3300
@@
 $EndComp
 $Comp
-L Wheel_ECU-rescue:GND #PWR09
+L Motor_ECU-rescue:GND-Wheel_ECU-rescue #PWR09
 U 1 1 5BFC312E
 P 8650 1900
@@
 $EndComp
 $Comp
-L Wheel_ECU-rescue:+5V #PWR010
+L Motor_ECU-rescue:+5V-Wheel_ECU-rescue #PWR010
 U 1 1 5BFC3169
 P 5650 2800
@@
 $EndComp
 $Comp
-L Wheel_ECU-rescue:+5V #PWR011
+L Motor_ECU-rescue:+5V-Wheel_ECU-rescue #PWR011
 U 1 1 5BFC31A4
 P 8200 1550
@@
 	7300 3000 7400 3000
 $Comp
-L Wheel_ECU-rescue:Conn_01x04 J1
+L Motor_ECU-rescue:Conn_01x04-Wheel_ECU-rescue J1
 U 1 1 5BFC3BD9
 P 10100 4400
@@
 $EndComp
 $Comp
-L Wheel_ECU-rescue:Conn_01x04 J2
+L Motor_ECU-rescue:Conn_01x04-Wheel_ECU-rescue J2
 U 1 1 5BFC3C20
 P 10100 5650
@@
 	9900 5650 9500 5650
 $Comp
-L Wheel_ECU-rescue:GND #PWR012
+L Motor_ECU-rescue:GND-Wheel_ECU-rescue #PWR012
 U 1 1 5BFC4380
 P 9800 4800
@@
 $EndComp
 $Comp
-L Wheel_ECU-rescue:+5V #PWR013
+L Motor_ECU-rescue:+5V-Wheel_ECU-rescue #PWR013
 U 1 1 5BFC43C1
 P 9150 4150
@@
 	2300 3700 2300 3600
 $Comp
-L Wheel_ECU-rescue:+5V #PWR014
+L Motor_ECU-rescue:+5V-Wheel_ECU-rescue #PWR014
 U 1 1 5BFCA92E
 P 10600 1650
@@
 	10600 1800 10600 1650
 $Comp
-L Wheel_ECU-rescue:GND #PWR015
+L Motor_ECU-rescue:GND-Wheel_ECU-rescue #PWR015
 U 1 1 5BFCAA26
 P 10250 2250
@@
 SWCLK
 $Comp
-L Wheel_ECU-rescue:GND #PWR016
+L Motor_ECU-rescue:GND-Wheel_ECU-rescue #PWR016
 U 1 1 5BFDD49A
 P 7100 2150
@@
 	7100 1700 7100 2150
 $Comp
-L Wheel_ECU-rescue:GND #PWR017
+L Motor_ECU-rescue:GND-Wheel_ECU-rescue #PWR017
 U 1 1 5BFDD5FE
 P 5500 2150
@@
 	5500 1800 5500 2150
 $Comp
-L Wheel_ECU-rescue:+5V #PWR018
+L Motor_ECU-rescue:+5V-Wheel_ECU-rescue #PWR018
 U 1 1 5BFDD7A5
 P 5500 1450
@@
 $EndComp
 $Comp
-L Wheel_ECU-rescue:+5V #PWR019
+L Motor_ECU-rescue:+5V-Wheel_ECU-rescue #PWR019
 U 1 1 5BFDD810
 P 7000 1450
@@
 	2500 6800 2400 6800
 $Comp
-L Wheel_ECU-rescue:C C6
+L Motor_ECU-rescue:C-Wheel_ECU-rescue C6
 U 1 1 5C004434
 P 950 4050
@@
 $EndComp
 $Comp
-L Wheel_ECU-rescue:C C7
+L Motor_ECU-rescue:C-Wheel_ECU-rescue C7
 U 1 1 5C0048A0
 P 1850 4050
@@
 Connection ~ 2450 3900
 $Comp
-L Wheel_ECU-rescue:C C9
+L Motor_ECU-rescue:C-Wheel_ECU-rescue C9
 U 1 1 5C005831
 P 1550 4050
@@
 $EndComp
 $Comp
-L Wheel_ECU-rescue:C C8
+L Motor_ECU-rescue:C-Wheel_ECU-rescue C8
 U 1 1 5C00587E
 P 1250 4050
@@
 Connection ~ 1250 3700
 $Comp
-L Wheel_ECU-rescue:+5V #PWR020
+L Motor_ECU-rescue:+5V-Wheel_ECU-rescue #PWR020
 U 1 1 5C03C916
 P 1350 1500
@@
 	1250 3700 1550 3700
 $Comp
-L wheel_ecu:IFX9201SG U1
+L motor_drivers:IFX9201SG U1
 U 1 1 5D08615A
 P 3150 1400
@@
 	5550 6300 4850 6300
 $Comp
-L Wheel_ECU-rescue:C C10
+L Motor_ECU-rescue:C-Wheel_ECU-rescue C10
 U 1 1 5D1439C8
 P 7900 5700
@@
 	7900 6000 8250 6000
 $Comp
-L Wheel_ECU-rescue:+5V #PWR01
+L Motor_ECU-rescue:+5V-Wheel_ECU-rescue #PWR01
 U 1 1 5D189F87
 P 7500 5350
@@
 $EndComp
 $Comp
-L Wheel_ECU-rescue:GND #PWR024
+L Motor_ECU-rescue:GND-Wheel_ECU-rescue #PWR024
 U 1 1 60286399
 P 6850 4950
@@
 	1050 1800 1050 1750
 $Comp
-L Wheel_ECU-rescue:C C14
+L Motor_ECU-rescue:C-Wheel_ECU-rescue C14
 U 1 1 6028D85A
 P 7200 4500
@@
 $EndComp
 $Comp
-L Wheel_ECU-rescue:C C13
+L Motor_ECU-rescue:C-Wheel_ECU-rescue C13
 U 1 1 6029F26A
 P 6850 4500
@@
 $EndComp
 $Comp
-L Wheel_ECU-rescue:C C11
+L Motor_ECU-rescue:C-Wheel_ECU-rescue C11
 U 1 1 6029FB2E
 P 3800 2850
@@
 $EndComp
 $Comp
-L Wheel_ECU-rescue:GND #PWR022
+L Motor_ECU-rescue:GND-Wheel_ECU-rescue #PWR022
 U 1 1 602A1AE9
 P 4000 3100
@@
 $EndComp
 $Comp
-L Wheel_ECU-rescue:C C12
+L Motor_ECU-rescue:C-Wheel_ECU-rescue C12
 U 1 1 602A1E6A
 P 4150 2850
@@
 	7200 4300 7600 4300
 $Comp
-L Wheel_ECU-rescue:TVS_Diode D2
+L Motor_ECU-rescue:TVS_Diode-Wheel_ECU-rescue D2
 U 1 1 60487B60
 P 6800 4900
@@
 	6850 4900 6850 4700
 $Comp
-L Wheel_ECU-rescue:+5V #PWR025
+L Motor_ECU-rescue:+5V-Wheel_ECU-rescue #PWR025
 U 1 1 6034D88D
 P 850 2750
@@
 Connection ~ 6000 3150
 $Comp
-L Wheel_ECU-rescue:GND #PWR027
+L Motor_ECU-rescue:GND-Wheel_ECU-rescue #PWR027
 U 1 1 603AB356
 P 9350 3600
@@
 $EndComp
 $Comp
-L Wheel_ECU-rescue:+5V #PWR026
+L Motor_ECU-rescue:+5V-Wheel_ECU-rescue #PWR026
 U 1 1 603AB7F6
 P 9350 2800

Commit message: Replace the 4-pin connectors with the new 5-pin connector
Parts:
- removed J5: Conn_01x02, Connector_PinHeader_2.54mm:PinHeader_1x02_P2.54mm_Vertical, symbol Connector_Generic:Conn_01x02
- J1, J2: value Conn_01x04 -> Conn_01x05; footprint Pin_Headers:Pin_Header_Straight_1x04_Pitch2.54mm -> Connector_PinHeader_2.54mm:PinHeader_1x05_P2.54mm_Vertical; symbol Motor_ECU-rescue:Conn_01x04-Wheel_ECU-rescue -> Connector_Generic:Conn_01x05
Connections:
- net +5V: now also J1.4 (Pin_4), J2.4 (Pin_4); no longer J1.3 (Pin_3), J2.3 (Pin_3)
- net +BATT: now also J1.3 (Pin_3), J2.3 (Pin_3)
- net GND: now also J1.5 (Pin_5), J2.5 (Pin_5); no longer J1.4 (Pin_4), J2.4 (Pin_4)
Changed lines of the file:
@@
 Sheet 1 1
 Title "Wolley Motor ECU"
-Date "2021-02-12"
-Rev "1.0"
+Date "2022-02-12"
+Rev "1.4"
 Comp "Knekt Technologies AB"
 Comment1 ""
@@
 	1    0    0    -1
 $EndComp
-Text GLabel 9850 5550 0    60   Input ~ 0
+Text GLabel 9850 5450 0    60   Input ~ 0
 CAN-
-Text GLabel 9500 5650 0    60   Input ~ 0
+Text GLabel 9500 5550 0    60   Input ~ 0
 CAN+
 $Comp
@@
 L Motor_ECU-rescue:+5V-Wheel_ECU-rescue #PWR07
 U 1 1 5BFC2D01
-P 9150 5400
-F 0 "#PWR07" H 9150 5250 50  0001 C CNN
-F 1 "+5V" H 9150 5540 50  0000 C CNN
-F 2 "" H 9150 5400 50  0001 C CNN
-F 3 "" H 9150 5400 50  0001 C CNN
-	1    9150 5400
+P 8900 5400
+F 0 "#PWR07" H 8900 5250 50  0001 C CNN
+F 1 "+5V" H 8900 5540 50  0000 C CNN
+F 2 "" H 8900 5400 50  0001 C CNN
+F 3 "" H 8900 5400 50  0001 C CNN
+	1    8900 5400
 	1    0    0    -1
 $EndComp
@@
 	7300 3000 7400 3000
 $Comp
-L Motor_ECU-rescue:Conn_01x04-Wheel_ECU-rescue J1
+L Connector_Generic:Conn_01x05 J1
 U 1 1 5BFC3BD9
 P 10100 4400
-F 0 "J1" H 10100 4600 50  0000 C CNN
-F 1 "Conn_01x04" H 10100 4100 50  0000 C CNN
-F 2 "Pin_Headers:Pin_Header_Straight_1x04_Pitch2.54mm" H 10100 4400 50  0001 C CNN
+F 0 "J1" H 10100 4700 50  0000 C CNN
+F 1 "Conn_01x05" H 10100 4100 50  0000 C CNN
+F 2 "Connector_PinHeader_2.54mm:PinHeader_1x05_P2.54mm_Vertical" H 10100 4400 50  0001 C CNN
 F 3 "" H 10100 4400 50  0001 C CNN
 	1    10100 4400
@@
 $EndComp
 $Comp
-L Motor_ECU-rescue:Conn_01x04-Wheel_ECU-rescue J2
+L Connector_Generic:Conn_01x05 J2
 U 1 1 5BFC3C20
 P 10100 5650
-F 0 "J2" H 10100 5850 50  0000 C CNN
-F 1 "Conn_01x04" H 10100 5350 50  0000 C CNN
-F 2 "Pin_Headers:Pin_Header_Straight_1x04_Pitch2.54mm" H 10100 5650 50  0001 C CNN
+F 0 "J2" H 10100 5950 50  0000 C CNN
+F 1 "Conn_01x05" H 10100 5350 50  0000 C CNN
+F 2 "Connector_PinHeader_2.54mm:PinHeader_1x05_P2.54mm_Vertical" H 10100 5650 50  0001 C CNN
 F 3 "" H 10100 5650 50  0001 C CNN
 	1    10100 5650
 	1    0    0    -1
 $EndComp
-Wire Wire Line
-	9900 5550 9850 5550
-Wire Wire Line
-	9900 5650 9500 5650
 $Comp
 L Motor_ECU-rescue:GND-Wheel_ECU-rescue #PWR012
@@
 L Motor_ECU-rescue:+5V-Wheel_ECU-rescue #PWR013
 U 1 1 5BFC43C1
-P 9150 4150
-F 0 "#PWR013" H 9150 4000 50  0001 C CNN
-F 1 "+5V" H 9150 4290 50  0000 C CNN
-F 2 "" H 9150 4150 50  0001 C CNN
-F 3 "" H 9150 4150 50  0001 C CNN
-	1    9150 4150
+P 8900 4150
+F 0 "#PWR013" H 8900 4000 50  0001 C CNN
+F 1 "+5V" H 8900 4290 50  0000 C CNN
+F 2 "" H 8900 4150 50  0001 C CNN
+F 3 "" H 8900 4150 50  0001 C CNN
+	1    8900 4150
 	1    0    0    -1
 $EndComp
 Wire Wire Line
 	9900 4600 9800 4600
-Text GLabel 9850 4300 0    60   Output ~ 0
+Text GLabel 9850 4200 0    60   Output ~ 0
 CAN-
-Text GLabel 9500 4400 0    60   Output ~ 0
+Text GLabel 9500 4300 0    60   Output ~ 0
 CAN+
-Wire Wire Line
-	9900 4400 9500 4400
-Wire Wire Line
-	9900 4300 9850 4300
 Text GLabel 10100 1500 2    60   Input ~ 0
 CAN+
@@
 $EndComp
 $Comp
-L Connector_Generic:Conn_01x02 J5
-U 1 1 6027FA18
-P 7800 4300
-F 0 "J5" H 7880 4292 50  0000 L CNN
-F 1 "Conn_01x02" H 7880 4201 50  0000 L CNN
-F 2 "Connector_PinHeader_2.54mm:PinHeader_1x02_P2.54mm_Vertical" H 7800 4300 50  0001 C CNN
-F 3 "~" H 7800 4300 50  0001 C CNN
-	1    7800 4300
-	1    0    0    -1
-$EndComp
-$Comp
 L Motor_ECU-rescue:GND-Wheel_ECU-rescue #PWR024
 U 1 1 60286399
@@
 Wire Wire Line
 	6850 4300 6850 4350
-Connection ~ 7200 4300
 Wire Wire Line
 	6850 4950 6850 4900
@@
 Wire Wire Line
 	6850 4700 6850 4650
-Connection ~ 7200 4700
 Wire Wire Line
 	6850 4200 6850 4300
@@
 	9800 4600 9800 4800
 Wire Wire Line
-	9900 4500 9150 4500
-Wire Wire Line
-	9150 4500 9150 4150
-Wire Wire Line
-	9900 5750 9150 5750
-Wire Wire Line
-	9150 5750 9150 5400
+	9900 4500 8900 4500
+Wire Wire Line
+	9900 5750 8900 5750
+Wire Wire Line
+	8900 5750 8900 5400
 Wire Wire Line
 	9750 6000 9750 5850
 Wire Wire Line
 	9750 5850 9900 5850
-Wire Wire Line
-	7500 4700 7200 4700
-Wire Wire Line
-	7500 4700 7500 4400
-Wire Wire Line
-	7500 4400 7600 4400
-Wire Wire Line
-	7200 4300 7600 4300
 $Comp
 L Motor_ECU-rescue:TVS_Diode-Wheel_ECU-rescue D2
@@
 Wire Wire Line
 	2500 5500 2400 5500
+$Comp
+L power:+BATT #PWR0101
+U 1 1 61E545A8
+P 9050 4350
+F 0 "#PWR0101" H 9050 4200 50  0001 C CNN
+F 1 "+BATT" H 9065 4523 50  0000 C CNN
+F 2 "" H 9050 4350 50  0001 C CNN
+F 3 "" H 9050 4350 50  0001 C CNN
+	1    9050 4350
+	1    0    0    -1
+$EndComp
+Wire Wire Line
+	8900 4150 8900 4500
+Wire Wire Line
+	9500 4300 9900 4300
+Wire Wire Line
+	9900 4200 9850 4200
+Wire Wire Line
+	9050 4400 9050 4350
+Wire Wire Line
+	9050 4400 9900 4400
+$Comp
+L power:+BATT #PWR0102
+U 1 1 61E8CB9F
+P 9050 5600
+F 0 "#PWR0102" H 9050 5450 50  0001 C CNN
+F 1 "+BATT" H 9065 5773 50  0000 C CNN
+F 2 "" H 9050 5600 50  0001 C CNN
+F 3 "" H 9050 5600 50  0001 C CNN
+	1    9050 5600
+	1    0    0    -1
+$EndComp
+Wire Wire Line
+	9050 5650 9050 5600
+Wire Wire Line
+	9050 5650 9900 5650
+Wire Wire Line
+	9500 5550 9900 5550
+Wire Wire Line
+	9900 5450 9850 5450
 $EndSCHEMATC
